Commit message: Add nvidia jetson to go1 urdf

File: urdf/go1.urdf (robot description, URDF)
Before this commit: robot go1, 52 links, 51 joints
Links:
- removed link rs_lidar
- added link nvidia, mass 1e-5; collision box size=0.1 0.1 0.07; visual mesh filename=package://rm3100_driver/urdf/meshes/nvidia-agx-orin-dev-kit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 scale=1 1 1
- added link rslidar, mass 1e-5; collision cylinder length=0.1 radius=0.05; visual mesh filename=package://rm3100_driver/urdf/meshes/bpearl.dae scale=1 1 1
Joints:
- added joint nvidia_joint: type fixed, parent trunk, child nvidia, origin xyz=-0.05 -0.05 0.12 rpy=0 0 0
- joint laser_joint: child rs_lidar -> rslidar

Commit message: Last version urdf, Add RM3100 driver and startup.sh, Update README

File: urdf/go1.urdf (robot description, URDF)
Before this commit: robot go1, 53 links, 52 joints
Links:
- added link rslidar_main
Joints:
- added joint laser_main_joint: type fixed, parent trunk, child rslidar_main, origin xyz=0.178 -0.02 0.211 rpy=0 1.57 0
- joint floating_base: origin xyz=0 0 0 rpy=0 0 0 -> xyz=0 0 0 rpy=0 0 1.57
- joint laser_joint: origin xyz=0.178 0 0.211 rpy=-1.57 1.57 0 -> xyz=0 0 0 rpy=0 0 0.02; parent trunk -> rslidar_main
- joint realsense_joint: origin xyz=0.177033 0 0.129929 rpy=-1.57 0 1.57 -> xyz=0.177033 0 0.129929 rpy=0 0 0
