Commit message: Add Hesai-JT128 to URDF and meshes.

File: ros2_ws/go1_description/urdf/go1.urdf (robot description, URDF)
Before this commit: robot go1, 54 links, 53 joints
Links:
- removed link rslidar
- removed link rslidar_main
- added link hesai
- added link hesai_jt128, mass 1e-5; collision cylinder length=0.08 radius=0.035; visual mesh filename=package://go1_description/meshes/hesai-jt128.dae scale=0.001 0.001 0.001
Joints:
- removed joint laser_joint
- removed joint laser_main_joint
- added joint hesai_joint: type fixed, parent hesai, child hesai_jt128, origin xyz=0 0 0 rpy=0 0 0.02
- added joint hesai_main_joint: type fixed, parent trunk, child hesai, origin xyz=0.168 -0.02 0.211 rpy=0 1.57 0

Commit message: Add Lidar support meshes and URDF. Hesai - Realsense calibration

File: ros2_ws/go1_description/urdf/go1.urdf (robot description, URDF)
Before this commit: robot go1, 54 links, 53 joints
Links:
- removed link hesai_jt128
- added link hesai_lidar, mass 1e-5; collision cylinder length=0.08 radius=0.035; visual mesh filename=package://go1_description/meshes/hesai-jt128.dae scale=0.001 0.001 0.001
- link support_link: geometry collision cylinder length=0.2 radius=0.04; visual mesh filename=package://go1_description/meshes/Suporte_Lidar_V006.dae scale=1 1 1
Joints:
- joint hesai_joint: child hesai_jt128 -> hesai_lidar; origin xyz=0 0 0 rpy=0 0 0.02 -> xyz=0 0 0 rpy=0 0 2
- joint hesai_main_joint: origin xyz=0.168 -0.02 0.211 rpy=0 1.57 0 -> xyz=0.175 -0.02 0.1885 rpy=0.0 1.57 0.0
